Commit message: housekeeping for final proj

File: body.urdf (robot description, URDF)
Before this commit: robot robot, 3 links, 2 joints
Links:
- added link BackLowerLeg, mass 1; collision box size=0.2 0.2 1.0; visual box size=0.2 0.2 1.0
- added link FrontLowerLeg, mass 1; collision box size=0.2 0.2 1.0; visual box size=0.2 0.2 1.0
- added link LeftLeg, mass 1; collision box size=1.0 0.2 0.2; visual box size=1.0 0.2 0.2
- added link LeftLowerLeg, mass 1; collision box size=0.2 0.2 1.0; visual box size=0.2 0.2 1.0
- added link RightLeg, mass 1; collision box size=1.0 0.2 0.2; visual box size=1.0 0.2 0.2
- added link RightLowerLeg, mass 1; collision box size=0.2 0.2 1.0; visual box size=0.2 0.2 1.0
- link BackLeg: geometry collision box size=0.2 1.0 0.2; visual box size=0.2 1.0 0.2
- link FrontLeg: geometry collision box size=0.2 1.0 0.2; visual box size=0.2 1.0 0.2
Joints:
- added joint BackLeg_BackLowerLeg: type revolute, parent BackLeg, child BackLowerLeg, origin xyz=0 -1.0 0 rpy=0 0 0, axis 1 0 0, limit lower=-0.6 upper=0.6 effort=100 velocity=1.0
- added joint FrontLeg_FrontLowerLeg: type revolute, parent FrontLeg, child FrontLowerLeg, origin xyz=0 1.0 0 rpy=0 0 0, axis 1 0 0, limit lower=-0.6 upper=0.6 effort=100 velocity=1.0
- added joint LeftLeg_LeftLowerLeg: type revolute, parent LeftLeg, child LeftLowerLeg, origin xyz=-1.0 0 0 rpy=0 0 0, axis 0 1 0, limit lower=-0.6 upper=0.6 effort=100 velocity=1.0
- added joint RightLeg_RightLowerLeg: type revolute, parent RightLeg, child RightLowerLeg, origin xyz=1.0 0 0 rpy=0 0 0, axis 0 1 0, limit lower=-0.6 upper=0.6 effort=100 velocity=1.0
- added joint Torso_LeftLeg: type revolute, parent Torso, child LeftLeg, origin xyz=-0.5 0 1.0 rpy=0 0 0, axis 0 1 0, limit lower=-0.6 upper=0.6 effort=100 velocity=1.0
- added joint Torso_RightLeg: type revolute, parent Torso, child RightLeg, origin xyz=0.5 0 1.0 rpy=0 0 0, axis 0 1 0, limit lower=-0.6 upper=0.6 effort=100 velocity=1.0
- joint Torso_BackLeg: axis 0 1 0 -> 1 0 0; limit lower=-3.14159 upper=3.14159 effort=0.0 velocity=0.0 -> lower=-0.6 upper=0.6 effort=100 velocity=1.0; origin xyz=1.0 0 1.0 rpy=0 0 0 -> xyz=0 -0.5 1.0 rpy=0 0 0
- joint Torso_FrontLeg: axis 0 1 0 -> 1 0 0; limit lower=-3.14159 upper=3.14159 effort=0.0 velocity=0.0 -> lower=-0.6 upper=0.6 effort=100 velocity=1.0; origin xyz=2.0 0 1.0 rpy=0 0 0 -> xyz=0 0.5 1.0 rpy=0 0 0

Commit message: milestone1 final proj complete

File: body.urdf (robot description, URDF)
Before this commit: robot robot, 9 links, 8 joints
Links:
- removed link BackLowerLeg
- removed link FrontLowerLeg
- removed link LeftLeg
- removed link LeftLowerLeg
- removed link RightLeg
- removed link RightLowerLeg
- link BackLeg: geometry collision box size=1 1 1; visual box size=1 1 1
- link FrontLeg: geometry collision box size=1 1 1; visual box size=1 1 1
Joints:
- removed joint BackLeg_BackLowerLeg
- removed joint FrontLeg_FrontLowerLeg
- removed joint LeftLeg_LeftLowerLeg
- removed joint RightLeg_RightLowerLeg
- removed joint Torso_LeftLeg
- removed joint Torso_RightLeg
- joint Torso_BackLeg: limit lower=-0.6 upper=0.6 effort=100 velocity=1.0 -> lower=-3.14159 upper=3.14159 effort=0.0 velocity=0.0; origin xyz=0 -0.5 1.0 rpy=0 0 0 -> xyz=1.0 0 1.0 rpy=0 0 0
- joint Torso_FrontLeg: limit lower=-0.6 upper=0.6 effort=100 velocity=1.0 -> lower=-3.14159 upper=3.14159 effort=0.0 velocity=0.0; origin xyz=0 0.5 1.0 rpy=0 0 0 -> xyz=2.0 0 1.0 rpy=0 0 0
